Commit message: add collision mass and inertia

File: src/fishbot_description/urdf/actuator/caster.urdf.xacro (robot description, xacro)
@@ -1,4 +1,5 @@
 <?xml version="1.0"?>
 <robot xmlns:xacro="http://www.ros.org/wiki/xacro">
+    <xacro:include filename="$(find fishbot_description)/urdf/common_inertia.xacro"/>
     <xacro:macro name="caster_xacro" params="caster_name xyz">
         <link name="${caster_name}_link">
@@ -12,4 +13,14 @@
                 </material>
             </visual>
+            <collision>
+                <origin xyz="0.0 0.0 0.0" rpy="0.0 0.0 0.0"/>
+                <geometry>
+                    <sphere radius="0.016"/>
+                </geometry>
+                <material name="yellow">
+                    <color rgba="1.0 1.0 0.0 0.8"/>
+                </material>
+            </collision>
+            <xacro:sphere_inertia m="0.05" r="0.016"/>
         </link>
         <joint name="${caster_name}_joint" type="fixed">

File: src/fishbot_description/urdf/actuator/wheel.urdf.xacro (robot description, xacro)
@@ -1,4 +1,5 @@
 <?xml version="1.0"?>
 <robot xmlns:xacro="http://www.ros.org/wiki/xacro">
+    <xacro:include filename="$(find fishbot_description)/urdf/common_inertia.xacro"/>
     <xacro:macro name="wheel_xacro" params="wheel_name xyz">
         <link name="${wheel_name}_link">
@@ -12,4 +13,14 @@
                 </material>
             </visual>
+            <collision>
+                <origin xyz="0.0 0.0 0.0" rpy="1.57079 0.0 0.0"/>
+                <geometry>
+                    <cylinder radius="0.032" length="0.04"/>>
+                </geometry>
+                <material name="yellow">
+                    <color rgba="1.0 1.0 0.0 0.8"/>
+                </material>
+            </collision>
+            <xacro:cylinder_inertia m="0.05" r="0.032" h="0.04"/>
         </link>
         <joint name="${wheel_name}_joint" type="continuous">

File: src/fishbot_description/urdf/base.urdf.xacro (robot description, xacro)
@@ -1,16 +1,34 @@
 <?xml version="1.0"?>
 <robot xmlns:xacro="http://www.ros.org/wiki/xacro">
+    <xacro:include filename="$(find fishbot_description)/urdf/common_inertia.xacro"/>
     <xacro:macro name="base_xacro" params="length radius">
+        <link name="base_footprint">
+        </link>
         <link name="base_link">
-        <visual>
-            <origin xyz="0.0 0.0 0.0" rpy="0.0 0.0 0.0"/>
-            <geometry>
-            <cylinder radius="${radius}" length="${length}"/>
-            </geometry>
-            <material name="white">
-            <color rgba="1.0 1.0 1.0 0.5"/>
-            </material>
-        </visual>
+            <visual>
+                <origin xyz="0.0 0.0 0.0" rpy="0.0 0.0 0.0"/>
+                <geometry>
+                <cylinder radius="${radius}" length="${length}"/>
+                </geometry>
+                <material name="white">
+                <color rgba="1.0 1.0 1.0 0.5"/>
+                </material>
+            </visual>
+            <collision>
+                <origin xyz="0.0 0.0 0.0" rpy="0.0 0.0 0.0"/>
+                <geometry>
+                <cylinder radius="${radius}" length="${length}"/>
+                </geometry>
+                <material name="white">
+                <color rgba="1.0 1.0 1.0 0.5"/>
+                </material>
+            </collision>
+            <xacro:cylinder_inertia m="1.0" r="${radius}" h="${length}"/>
         </link>
+        <joint name="joint_name" type="fixed">
+            <origin xyz="0.0 0.0 ${length/2.0+0.032-0.001}" rpy="0.0 0.0 0.0"/>
+            <parent link="base_footprint"/>
+            <child link="base_link"/>
+        </joint>
     </xacro:macro>
 </robot>

File: src/fishbot_description/urdf/sensor/camera.urdf.xacro (robot description, xacro)
@@ -1,15 +1,26 @@
 <?xml version="1.0"?>
 <robot xmlns:xacro="http://www.ros.org/wiki/xacro">
+    <xacro:include filename="$(find fishbot_description)/urdf/common_inertia.xacro"/>
     <xacro:macro name="camera_xacro" params="xyz">
         <link name="camera_link">
-        <visual>
-            <origin xyz="0.0 0.0 0.0" rpy="0.0 0.0 0.0"/>
-            <geometry>
-            <box size="0.02 0.10 0.02"/>
-            </geometry>
-            <material name="black">
-            <color rgba="0.0 0.0 0.0 0.5"/>
-            </material>
-        </visual>
+            <visual>
+                <origin xyz="0.0 0.0 0.0" rpy="0.0 0.0 0.0"/>
+                <geometry>
+                    <box size="0.02 0.10 0.02"/>
+                </geometry>
+                <material name="black">
+                    <color rgba="0.0 0.0 0.0 0.5"/>
+                </material>
+            </visual>
+            <collision>
+                <origin xyz="0.0 0.0 0.0" rpy="0.0 0.0 0.0"/>
+                <geometry>
+                    <box size="0.02 0.10 0.02"/>
+                </geometry>
+                <material name="black">
+                    <color rgba="0.0 0.0 0.0 0.5"/>
+                </material>
+            </collision>
+            <xacro:box_inertia m="0.1" w="0.02" h="0.10" d="0.02"/>
         </link>
         <joint name="camera_joint" type="fixed">

File: src/fishbot_description/urdf/sensor/imu.urdf.xacro (robot description, xacro)
@@ -1,15 +1,26 @@
 <?xml version="1.0"?>
 <robot xmlns:xacro="http://www.ros.org/wiki/xacro">
+    <xacro:include filename="$(find fishbot_description)/urdf/common_inertia.xacro"/>
     <xacro:macro name="imu_xacro" params="xyz">
         <link name="imu_link">
-        <visual>
-            <origin xyz="0.0 0.0 0.0" rpy="0.0 0.0 0.0"/>
-            <geometry>
-            <box size="0.02 0.02 0.02"/>
-            </geometry>
-            <material name="black">
-            <color rgba="0.0 0.0 0.0 0.5"/>
-            </material>
-        </visual>
+            <visual>
+                <origin xyz="0.0 0.0 0.0" rpy="0.0 0.0 0.0"/>
+                <geometry>
+                <box size="0.02 0.02 0.02"/>
+                </geometry>
+                <material name="black">
+                <color rgba="0.0 0.0 0.0 0.5"/>
+                </material>
+            </visual>
+            <collision>
+                <origin xyz="0.0 0.0 0.0" rpy="0.0 0.0 0.0"/>
+                <geometry>
+                <box size="0.02 0.02 0.02"/>
+                </geometry>
+                <material name="black">
+                <color rgba="0.0 0.0 0.0 0.5"/>
+                </material>
+            </collision>
+            <xacro:box_inertia m="0.05" w="0.02" h="0.02" d="0.02"/>
         </link>
         <joint name="imu_joint" type="fixed">

File: src/fishbot_description/urdf/sensor/laser.urdf.xacro (robot description, xacro)
@@ -1,4 +1,5 @@
 <?xml version="1.0"?>
 <robot xmlns:xacro="http://www.ros.org/wiki/xacro">
+    <xacro:include filename="$(find fishbot_description)/urdf/common_inertia.xacro"/>
     <xacro:macro name="laser_xacro" params="xyz">
         <link name="laser_cylinder_link">
@@ -12,4 +13,14 @@
                 </material>
             </visual>
+            <collision>
+                <origin xyz="0.0 0.0 0.0" rpy="0.0 0.0 0.0"/>
+                <geometry>
+                    <cylinder radius="0.01" length="0.10"/>
+                </geometry>
+                <material name="black">
+                <color rgba="0.0 0.0 0.0 1.0"/>
+                </material>
+            </collision>
+            <xacro:cylinder_inertia m="0.05" r="0.01" h="0.10"/>
         </link>
         <link name="laser_link">
@@ -23,4 +34,14 @@
                 </material>
             </visual>
+            <collision>
+                <origin xyz="0.0 0.0 0.0" rpy="0.0 0.0 0.0"/>
+                <geometry>
+                    <cylinder radius="0.02" length="0.02"/>
+                </geometry>
+                <material name="black">
+                <color rgba="0.0 0.0 0.0 1.0"/>
+                </material>
+            </collision>
+            <xacro:cylinder_inertia m="0.10" r="0.02" h="0.02"/>
         </link>
         <joint name="laser_joint" type="fixed">

Commit message: diff plugin control robot

File: src/fishbot_description/urdf/actuator/caster.urdf.xacro (robot description, xacro)
@@ -29,4 +29,17 @@
             <origin xyz="${xyz}" rpy="0.0 0.0 0.0"/>
         </joint>
+        <gazebo reference="${caster_name}_link">
+            <material>
+                Gazebo/Yellow
+            </material>
+            <!-- 切向摩擦系数 -->
+            <mu1 value="0.0"/>
+            <!-- 法向摩擦系数 -->
+            <mu2 value="0.0"/>
+            <!-- 接触刚度系数 -->
+            <kp value="1000000000.0"/>
+            <!-- 阻尼系数 -->
+            <kd value="1.0"/>
+        </gazebo>
     </xacro:macro>
 </robot>

File: src/fishbot_description/urdf/actuator/wheel.urdf.xacro (robot description, xacro)
@@ -30,4 +30,17 @@
             <axis xyz="0.0 1.0 0.0"/>
         </joint>
+        <gazebo reference="${wheel_name}_link">
+            <material>
+                Gazebo/Yellow
+            </material>
+            <!-- 切向摩擦系数 -->
+            <mu1 value="20.0"/>
+            <!-- 法向摩擦系数 -->
+            <mu2 value="20.0"/>
+            <!-- 接触刚度系数 -->
+            <kp value="1000000000.0"/>
+            <!-- 阻尼系数 -->
+            <kd value="1.0"/>
+        </gazebo>
     </xacro:macro>
 </robot>

File: src/fishbot_description/urdf/fishbot.urdf.xacro (robot description, xacro)
@@ -7,4 +7,5 @@
 <xacro:include filename="$(find fishbot_description)/urdf/actuator/wheel.urdf.xacro"/>
 <xacro:include filename="$(find fishbot_description)/urdf/actuator/caster.urdf.xacro"/>
+<xacro:include filename="$(find fishbot_description)/urdf/plugin/gazebo_control_plugin.xacro"/>
 <xacro:base_xacro length="0.12" radius="0.10"/>
 <xacro:imu_xacro xyz="0.0 0.0 0.02"/>
@@ -15,3 +16,4 @@
 <xacro:caster_xacro caster_name="front_caster" xyz="0.08 0.0 -0.076"/>
 <xacro:caster_xacro caster_name="rear_caster" xyz="-0.08 0.0 -0.076"/>
+<xacro:gazebo_control_plugin/>
 </robot>

File: src/fishbot_description/urdf/sensor/laser.urdf.xacro (robot description, xacro)
@@ -55,4 +55,14 @@
             <origin xyz="${xyz}" rpy="0.0 0.0 0.0"/>
         </joint>
+        <gazebo reference="laser_cylinder_link">
+            <material>
+                Gazebo/Black
+            </material>
+        </gazebo>
+        <gazebo reference="laser_link">
+            <material>
+                Gazebo/Black
+            </material>
+        </gazebo>
     </xacro:macro>
 </robot>
