Commit message: add lots of sensors like lidar, imu, point cloud

File: src/fishbot_description/urdf/fishbot.urdf.xacro (robot description, xacro)
@@ -8,4 +8,5 @@
 <xacro:include filename="$(find fishbot_description)/urdf/actuator/caster.urdf.xacro"/>
 <xacro:include filename="$(find fishbot_description)/urdf/plugin/gazebo_control_plugin.xacro"/>
+<xacro:include filename="$(find fishbot_description)/urdf/plugin/gazebo_sensor_plugin.xacro"/>
 <xacro:base_xacro length="0.12" radius="0.10"/>
 <xacro:imu_xacro xyz="0.0 0.0 0.02"/>
@@ -17,3 +18,4 @@
 <xacro:caster_xacro caster_name="rear_caster" xyz="-0.08 0.0 -0.076"/>
 <xacro:gazebo_control_plugin/>
+<xacro:gazebo_sensor_plugin/>
 </robot>

File: src/fishbot_description/urdf/sensor/camera.urdf.xacro (robot description, xacro)
@@ -24,4 +24,5 @@
             <xacro:box_inertia m="0.1" w="0.02" h="0.10" d="0.02"/>
         </link>
+        <link name="camera_optical_link"> </link>
         <joint name="camera_joint" type="fixed">
             <parent link="base_link"/>
@@ -29,4 +30,10 @@
             <origin xyz="${xyz}" rpy="0.0 0.0 0.0"/>
         </joint>
+        <joint name="camera_optical_joint" type="fixed">
+            <parent link="camera_link"/>
+                <child link="camera_optical_link"/>
+            <!-- <origin xyz="0.0 0.0 0.0" rpy="${-pi/2} 0.0 ${-pi/2}"/> -->
+                <origin xyz="0.0 0.0 0.0" rpy="0 0.0 0"/>
+        </joint>
     </xacro:macro>
 </robot>
