Commit message: fix a navigation bug

File: src/fishbot_description/urdf/base.urdf.xacro (robot description, xacro)
@@ -11,6 +11,6 @@
                 <cylinder radius="${radius}" length="${length}"/>
                 </geometry>
-                <material name="white">
-                <color rgba="1.0 1.0 1.0 0.5"/>
+                <material name="blue">
+                <color rgba="0.1 0.1 1.0 0.5"/>
                 </material>
             </visual>
@@ -20,11 +20,11 @@
                 <cylinder radius="${radius}" length="${length}"/>
                 </geometry>
-                <material name="white">
-                <color rgba="1.0 1.0 1.0 0.5"/>
+                <material name="blue">
+                <color rgba="0.1 0.1 1.0 0.5"/>
                 </material>
             </collision>
             <xacro:cylinder_inertia m="1.0" r="${radius}" h="${length}"/>
         </link>
-        <joint name="joint_name" type="fixed">
+        <joint name="base_joint" type="fixed">
             <origin xyz="0.0 0.0 ${length/2.0+0.032-0.001}" rpy="0.0 0.0 0.0"/>
             <parent link="base_footprint"/>

File: src/fishbot_description/urdf/fishbot.ros2_control.xacro (robot description, xacro)
@@ -37,5 +37,5 @@
                 <parameters>$(find fishbot_description)/config/fishbot_ros2_controller.yaml</parameters>
                 <ros>
-                    <remapping>/diff_drive_controller/odom:=/odometry</remapping>
+                    <remapping>/diff_drive_controller/odom:=/odom</remapping>
                     <remapping>/diff_drive_controller/cmd_vel:=/cmd_vel</remapping>
                 </ros>
